Commit message: s

File: PyBullet_test/Code/utils/internet robot/simple_plane - Copy.urdf (robot description, URDF)
Before this commit: robot custom_box, 1 links, 0 joints
Links:
- removed link box
- added link planeLink, mass .0; collision box size=30 30 10; visual mesh filename=plane_transparent.obj scale=1 1 1

File: PyBullet_test/Code/utils/internet robot/simple_plane.urdf (robot description, URDF)
Before this commit: robot track_environment, 1 links, 0 joints
Links:
- link plane_link: geometry collision box size=10 10 10; visual box size=10 10 10
